Commit message: arduino communication implemented. ready for test with sbc and lidar

File: urdf/olaf_copy.urdf (robot description, URDF)
Before this commit: robot olaf, 7 links, 6 joints
Joints:
- added joint base_footprint_joint: type fixed, parent base_footprint, child base_link, origin xyz=0.0 0.0 0.12 rpy=0.0 0.0 0.0
